File: Hardware/SAMD51_Thing_Plus.sch (EAGLE design)
At the start: 55 parts, among them J6 AMP FCI 10103594-0001LF, Q1 2.5A/30V, U1 MCP73831, U2 ATSAMD51J20A-A, U3 AP2112K-3.3V, U4 4MB Flash, Y1 32.768kHz

Commit message: engineer run of checklist-REDS
Parts:
- added U$69: QWIIC_LOGO_5MM, SparkFun-Aesthetics:QWIIC_LOGO_5MM
- C13, C19, C6: device SparkFun-Capacitors:4.7UF0603 -> SparkFun-Capacitors:4.7UF-0603-6.3V-(10%)
- D2: value BAT20J -> 1A/23V/620mV
Other:
- note added: "v10"
- note removed: "v03"
Changed lines of the file:
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@@
 <part name="GND11" library="SparkFun-Aesthetics" deviceset="GND" device=""/>
 <part name="GND12" library="SparkFun-Aesthetics" deviceset="GND" device=""/>
-<part name="C6" library="SparkFun-Capacitors" deviceset="4.7UF" device="0603" value="4.7uF"/>
-<part name="D2" library="SparkFun-DiscreteSemi" deviceset="DIODE-SCHOTTKY" device="-BAT20J" value="BAT20J"/>
+<part name="C6" library="SparkFun-Capacitors" deviceset="4.7UF" device="-0603-6.3V-(10%)" value="4.7uF"/>
+<part name="D2" library="SparkFun-DiscreteSemi" deviceset="DIODE-SCHOTTKY" device="-BAT20J" value="1A/23V/620mV"/>
 <part name="R7" library="SparkFun-Resistors" deviceset="10KOHM" device="-0603-1/10W-1%" value="10k"/>
 <part name="GND13" library="SparkFun-Aesthetics" deviceset="GND" device=""/>
@@
 <part name="SUPPLY25" library="SparkFun-Aesthetics" deviceset="V_BATT" device=""/>
 <part name="SUPPLY27" library="SparkFun-Aesthetics" deviceset="V_BATT" device=""/>
-<part name="C19" library="SparkFun-Capacitors" deviceset="4.7UF" device="0603" value="4.7uF"/>
+<part name="C19" library="SparkFun-Capacitors" deviceset="4.7UF" device="-0603-6.3V-(10%)" value="4.7uF"/>
 <part name="SUPPLY23" library="SparkFun-Aesthetics" deviceset="V_USB" device=""/>
 <part name="GND41" library="SparkFun-Aesthetics" deviceset="GND" device=""/>
@@
 <part name="C9" library="SparkFun-Capacitors" deviceset="0.1UF" device="-0402-16V-10%" value="0.1uF"/>
 <part name="SUPPLY13" library="SparkFun-PowerSymbols" deviceset="VCC" device=""/>
-<part name="C13" library="SparkFun-Capacitors" deviceset="4.7UF" device="0603" value="4.7uF"/>
+<part name="C13" library="SparkFun-Capacitors" deviceset="4.7UF" device="-0603-6.3V-(10%)" value="4.7uF"/>
 <part name="C14" library="SparkFun-Capacitors" deviceset="0.1UF" device="-0402-16V-10%" value="0.1uF"/>
 <part name="C15" library="SparkFun-Capacitors" deviceset="10UF" device="-0805-10V-10%" value="10uF"/>
@@
 <part name="H3" library="SparkFun-Hardware" deviceset="STAND-OFF" device=""/>
 <part name="H4" library="SparkFun-Hardware" deviceset="STAND-OFF" device=""/>
+<part name="U$69" library="SparkFun-Aesthetics" deviceset="QWIIC_LOGO" device="_5MM"/>
 </parts>
 <sheets>
@@
 <text x="200.66" y="63.5" size="2.54" layer="97" font="vector" align="top-left">GPIO13 LED</text>
 <text x="332.74" y="104.14" size="2.54" layer="97" font="vector" align="top-left">Headers</text>
-<text x="421.64" y="10.16" size="2.54" layer="94" font="vector" align="top-left">v03</text>
+<text x="421.64" y="10.16" size="2.54" layer="94" font="vector" align="top-left">v10</text>
 <text x="69.088" y="17.78" size="0.4064" layer="94" font="vector">C8 to be
 near U2.21</text>
@@
 <instance part="H3" gate="G$1" x="429.26" y="33.02"/>
 <instance part="H4" gate="G$1" x="429.26" y="30.48"/>
+<instance part="U$69" gate="G$1" x="300.228" y="3.81"/>
 </instances>
 <busses>
@@
 <pinref part="U4" gate="G$1" pin="!WP(D2)"/>
 <wire x1="355.6" y1="162.56" x2="355.6" y2="165.1" width="0.1524" layer="91"/>
-<wire x1="365.76" y1="139.7" x2="340.36" y2="139.7" width="0.1524" layer="91"/>
+<wire x1="368.3" y1="139.7" x2="340.36" y2="139.7" width="0.1524" layer="91"/>
 <wire x1="340.36" y1="139.7" x2="340.36" y2="162.56" width="0.1524" layer="91"/>
 <wire x1="340.36" y1="162.56" x2="355.6" y2="162.56" width="0.1524" layer="91"/>
@@
 <wire x1="403.86" y1="165.1" x2="403.86" y2="144.78" width="0.1524" layer="91"/>
 <pinref part="U4" gate="G$1" pin="VCC"/>
-<wire x1="403.86" y1="144.78" x2="401.32" y2="144.78" width="0.1524" layer="91"/>
+<wire x1="403.86" y1="144.78" x2="398.78" y2="144.78" width="0.1524" layer="91"/>
 <pinref part="U4" gate="G$1" pin="!HOLD(D3)"/>
-<wire x1="401.32" y1="142.24" x2="403.86" y2="142.24" width="0.1524" layer="91"/>
+<wire x1="398.78" y1="142.24" x2="403.86" y2="142.24" width="0.1524" layer="91"/>
 <wire x1="403.86" y1="142.24" x2="403.86" y2="144.78" width="0.1524" layer="91"/>
 <junction x="403.86" y="144.78"/>
@@
 <wire x1="363.22" y1="134.62" x2="363.22" y2="137.16" width="0.1524" layer="91"/>
 <pinref part="U4" gate="G$1" pin="GND"/>
-<wire x1="363.22" y1="137.16" x2="365.76" y2="137.16" width="0.1524" layer="91"/>
+<wire x1="363.22" y1="137.16" x2="368.3" y2="137.16" width="0.1524" layer="91"/>
 </segment>
 </net>
@@
 <segment>
 <pinref part="U4" gate="G$1" pin="SCK"/>
-<wire x1="401.32" y1="139.7" x2="403.86" y2="139.7" width="0.1524" layer="91"/>
+<wire x1="398.78" y1="139.7" x2="403.86" y2="139.7" width="0.1524" layer="91"/>
 <label x="403.86" y="139.7" size="1.27" layer="95" font="vector" xref="yes"/>
 </segment>
@@
 <segment>
 <pinref part="U4" gate="G$1" pin="SI(D0)"/>
-<wire x1="401.32" y1="137.16" x2="403.86" y2="137.16" width="0.1524" layer="91"/>
+<wire x1="398.78" y1="137.16" x2="403.86" y2="137.16" width="0.1524" layer="91"/>
 <label x="403.86" y="137.16" size="1.27" layer="95" font="vector" xref="yes"/>
 </segment>
@@
 <segment>
 <pinref part="U4" gate="G$1" pin="!CS"/>
-<wire x1="365.76" y1="144.78" x2="355.6" y2="144.78" width="0.1524" layer="91"/>
+<wire x1="368.3" y1="144.78" x2="355.6" y2="144.78" width="0.1524" layer="91"/>
 <wire x1="355.6" y1="144.78" x2="355.6" y2="149.86" width="0.1524" layer="91"/>
 <pinref part="R4" gate="G$1" pin="1"/>
@@
 <segment>
 <pinref part="U4" gate="G$1" pin="SO(D1)"/>
-<wire x1="365.76" y1="142.24" x2="363.22" y2="142.24" width="0.1524" layer="91"/>
+<wire x1="368.3" y1="142.24" x2="363.22" y2="142.24" width="0.1524" layer="91"/>
 <label x="363.22" y="142.24" size="1.27" layer="95" font="vector" rot="R180" xref="yes"/>
 </segment>
