File: Hardware/SAMD51_Thing_Plus.sch (EAGLE design)
At the start: 56 parts, among them J6 AMP FCI 10103594-0001LF, Q1 2.5A/30V, U1 MCP73831, U2 ATSAMD51J20A-A, U3 AP2112K-3.3V, U4 4MB Flash, Y1 32.768kHz

Commit message: Correct Label in Schematic
- The Dev board was incorrectly labeled as 4MB in the schematic. It is technically 4Mb after checking the BOM.
Parts:
- U4: value 4MB Flash -> 4Mb Flash
Changed lines of the file:
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@@
 <?xml version="1.0" encoding="utf-8"?>
 <!DOCTYPE eagle SYSTEM "eagle.dtd">
-<eagle version="9.1.0">
+<eagle version="7.6.0">
 <drawing>
 <settings>
 <setting alwaysvectorfont="no"/>
-<setting keepoldvectorfont="yes"/>
 <setting verticaltext="up"/>
 </settings>
@@
 <part name="TP1" library="SparkFun-Connectors" deviceset="TEST-POINT" device="TP_15TH_THRU"/>
 <part name="TP2" library="SparkFun-Connectors" deviceset="TEST-POINT" device="TP_15TH_THRU"/>
-<part name="U4" library="SparkFun-IC-Memory" deviceset="AT25SF041" device="" value="4MB Flash"/>
+<part name="U4" library="SparkFun-IC-Memory" deviceset="AT25SF041" device="" value="4Mb Flash"/>
 <part name="R4" library="SparkFun-Resistors" deviceset="10KOHM" device="-0603-1/10W-1%" value="10k"/>
 <part name="SUPPLY9" library="SparkFun-Aesthetics" deviceset="3.3V" device=""/>
